Commit message: updated the file pathing for the link meshes

File: simulation/isaac/assets/urdf/skeleton.urdf (robot description, URDF)
Before this commit: robot humanoid, 14 links, 13 joints
Links:
- link l_ankle_link: geometry collision mesh filename=../meshes/skeleton/l_ankle_link.stl; visual mesh filename=../meshes/skeleton/l_ankle_link.stl
- link l_foot_link: geometry collision mesh filename=../meshes/skeleton/l_foot_link.stl; visual mesh filename=../meshes/skeleton/l_foot_link.stl
- link l_hip_pitch_link: geometry collision mesh filename=../meshes/skeleton/l_hip_pitch_link.stl; visual mesh filename=../meshes/skeleton/l_hip_pitch_link.stl
- link l_hip_yaw_link: geometry collision mesh filename=../meshes/skeleton/l_hip_yaw_link.stl; visual mesh filename=../meshes/skeleton/l_hip_yaw_link.stl
- link l_shank_link: geometry collision mesh filename=../meshes/skeleton/l_shank_link.stl; visual mesh filename=../meshes/skeleton/l_shank_link.stl
- link l_thigh_link: geometry collision mesh filename=../meshes/skeleton/l_thigh_link.stl; visual mesh filename=../meshes/skeleton/l_thigh_link.stl
- link pelvis_link: geometry collision mesh filename=../meshes/skeleton/pelvis_link.stl; visual mesh filename=../meshes/skeleton/pelvis_link.stl
- link r_ankle_link: geometry collision mesh filename=../meshes/skeleton/r_ankle_link.stl; visual mesh filename=../meshes/skeleton/r_ankle_link.stl
- link r_foot_link: geometry collision mesh filename=../meshes/skeleton/r_foot_link.stl; visual mesh filename=../meshes/skeleton/r_foot_link.stl
- link r_hip_pitch_link: geometry collision mesh filename=../meshes/skeleton/r_hip_pitch_link.stl; visual mesh filename=../meshes/skeleton/r_hip_pitch_link.stl
- link r_hip_yaw_link: geometry collision mesh filename=../meshes/skeleton/r_hip_yaw_link.stl; visual mesh filename=../meshes/skeleton/r_hip_yaw_link.stl
- link r_shank_link: geometry collision mesh filename=../meshes/skeleton/r_shank_link.stl; visual mesh filename=../meshes/skeleton/r_shank_link.stl
- link r_thigh_link: geometry collision mesh filename=../meshes/skeleton/r_thigh_link.stl; visual mesh filename=../meshes/skeleton/r_thigh_link.stl
- link torso_link: geometry collision mesh filename=../meshes/skeleton/torso_link.stl; visual mesh filename=../meshes/skeleton/torso_link.stl

Commit message: cleaned up the formatting in skeleton.urdf file

File: simulation/isaac/assets/urdf/skeleton.urdf (robot description, URDF)
Before this commit: robot skeleton, 14 links, 13 joints
Links:
- link l_ankle_link: geometry collision mesh filename=../meshes/skeleton/collision_meshes/l_ankle_link_collision.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; visual mesh filename=../meshes/skeleton/l_ankle_link.stl
- link l_foot_link: geometry collision mesh filename=../meshes/skeleton/collision_meshes/l_foot_link_collision.s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; visual mesh filename=../meshes/skeleton/l_foot_link.stl
- link l_hip_pitch_link: geometry collision mesh filename=../meshes/skeleton/collision_meshes/l_hip_pitch_link_collis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; visual mesh filename=../meshes/skeleton/l_hip_pitch_link.stl
- link l_hip_yaw_link: geometry collision mesh filename=../meshes/skeleton/collision_meshes/l_hip_yaw_link_collisio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; visual mesh filename=../meshes/skeleton/l_hip_yaw_link.stl
- link l_shank_link: geometry collision mesh filename=../meshes/skeleton/collision_meshes/l_shank_link_collision.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; visual mesh filename=../meshes/skeleton/l_shank_link.stl
- link l_thigh_link: geometry collision mesh filename=../meshes/skeleton/collision_meshes/l_thigh_link_collision.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; visual mesh filename=../meshes/skeleton/l_thigh_link.stl
- link pelvis_link: geometry collision mesh filename=../meshes/skeleton/collision_meshes/pelvis_link_collision.s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; visual mesh filename=../meshes/skeleton/pelvis_link.stl
- link r_ankle_link: geometry collision mesh filename=../meshes/skeleton/collision_meshes/r_ankle_link_collision.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; visual mesh filename=../meshes/skeleton/r_ankle_link.stl
- link r_foot_link: geometry collision mesh filename=../meshes/skeleton/collision_meshes/r_foot_link_collision.s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; visual mesh filename=../meshes/skeleton/r_foot_link.stl
- link r_hip_pitch_link: geometry collision mesh filename=../meshes/skeleton/collision_meshes/r_hip_pitch_link_collis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; visual mesh filename=../meshes/skeleton/r_hip_pitch_link.stl
- link r_hip_yaw_link: geometry collision mesh filename=../meshes/skeleton/collision_meshes/r_hip_yaw_link_collisio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; visual mesh filename=../meshes/skeleton/r_hip_yaw_link.stl
- link r_shank_link: geometry collision mesh filename=../meshes/skeleton/collision_meshes/r_shank_link_collision.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; visual mesh filename=../meshes/skeleton/r_shank_link.stl
- link r_thigh_link: geometry collision mesh filename=../meshes/skeleton/collision_meshes/r_thigh_link_collision.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; visual mesh filename=../meshes/skeleton/r_thigh_link.stl
- link torso_link: geometry collision mesh filename=../meshes/skeleton/collision_meshes/torso_link_collision.stl; visual mesh filename=../meshes/skeleton/torso_link.stl

Commit message: URDF file configured for the robot link and joint placements.

File: simulation/isaac/assets/urdf/skeleton.urdf (robot description, URDF)
Before this commit: robot skeleton, 14 links, 13 joints
Links:
- removed link l_ankle_link
- removed link l_foot_link
- removed link l_hip_pitch_link
- removed link l_hip_yaw_link
- removed link l_shank_link
- removed link l_thigh_link
- removed link pelvis_link
- removed link r_ankle_link
- removed link r_foot_link
- removed link r_hip_pitch_link
- removed link r_hip_yaw_link
- removed link r_shank_link
- removed link r_thigh_link
- removed link torso_link
- added link robot_l_ankle_link, mass 2.497542686119488; collision mesh filename=meshes/robot_l_ankle_link.stl scale=0.001 0.001 0.001; visual mesh filename=meshes/robot_l_ankle_link.stl scale=0.001 0.001 0.001
- added link robot_l_foot_link, mass 2.78967156731517; collision mesh filename=meshes/robot_l_foot_link.stl scale=0.001 0.001 0.001; visual mesh filename=meshes/robot_l_foot_link.stl scale=0.001 0.001 0.001
- added link robot_l_hip_pitch_link, mass 2.4943200880759124; collision mesh filename=meshes/robot_l_hip_pitch_link.stl scale=0.001 0.001 0.001; visual mesh filename=meshes/robot_l_hip_pitch_link.stl scale=0.001 0.001 0.001
- added link robot_l_hip_yaw_link, mass 6.333603185323419; collision mesh filename=meshes/robot_l_hip_yaw_link.stl scale=0.001 0.001 0.001; visual mesh filename=meshes/robot_l_hip_yaw_link.stl scale=0.001 0.001 0.001
- added link robot_l_shank_link, mass 0.8515894596853654; collision mesh filename=meshes/robot_l_shank_link.stl scale=0.001 0.001 0.001; visual mesh filename=meshes/robot_l_shank_link.stl scale=0.001 0.001 0.001
- added link robot_l_thigh_link, mass 3.0917752218546957; collision mesh filename=meshes/robot_l_thigh_link.stl scale=0.001 0.001 0.001; visual mesh filename=meshes/robot_l_thigh_link.stl scale=0.001 0.001 0.001
- added link robot_pelvis_link, mass 0.4703666239440356; collision mesh filename=meshes/robot_pelvis_link.stl scale=0.001 0.001 0.001; visual mesh filename=meshes/robot_pelvis_link.stl scale=0.001 0.001 0.001
- added link robot_r_ankle_link, mass 2.4975426861194876; collision mesh filename=meshes/robot_r_ankle_link.stl scale=0.001 0.001 0.001; visual mesh filename=meshes/robot_r_ankle_link.stl scale=0.001 0.001 0.001
- added link robot_r_foot_link, mass 2.7896715673151693; collision mesh filename=meshes/robot_r_foot_link.stl scale=0.001 0.001 0.001; visual mesh filename=meshes/robot_r_foot_link.stl scale=0.001 0.001 0.001
- added link robot_r_hip_pitch_link, mass 2.4943200880759147; collision mesh filename=meshes/robot_r_hip_pitch_link.stl scale=0.001 0.001 0.001; visual mesh filename=meshes/robot_r_hip_pitch_link.stl scale=0.001 0.001 0.001
- added link robot_r_hip_yaw_link, mass 6.33360318547509; collision mesh filename=meshes/robot_r_hip_yaw_link.stl scale=0.001 0.001 0.001; visual mesh filename=meshes/robot_r_hip_yaw_link.stl scale=0.001 0.001 0.001
- added link robot_r_shank_link, mass 0.8515894596853654; collision mesh filename=meshes/robot_r_shank_link.stl scale=0.001 0.001 0.001; visual mesh filename=meshes/robot_r_shank_link.stl scale=0.001 0.001 0.001
- added link robot_r_thigh_link, mass 3.0917752218546957; collision mesh filename=meshes/robot_r_thigh_link.stl scale=0.001 0.001 0.001; visual mesh filename=meshes/robot_r_thigh_link.stl scale=0.001 0.001 0.001
- added link robot_torso_link, mass 3.4766230099551185; collision mesh filename=meshes/robot_torso_link.stl scale=0.001 0.001 0.001; visual mesh filename=meshes/robot_torso_link.stl scale=0.001 0.001 0.001
- added link world
Joints:
- removed joint l_ankle_joint
- removed joint l_foot_joint
- removed joint l_hip_pitch_joint
- removed joint l_hip_roll_joint
- removed joint l_hip_yaw_joint
- removed joint l_knee_joint
- removed joint r_ankle_joint
- removed joint r_foot_joint
- removed joint r_hip_pitch_joint
- removed joint r_hip_roll_joint
- removed joint r_hip_yaw_joint
- removed joint r_knee_joint
- removed joint torso_joint
- added joint robot_l_ankle_link_l_foot_joint: type continuous, parent robot_l_ankle_link, child robot_l_foot_link, origin xyz=0.07401155999999999 -5.9079999999998025e-05 0.009015649999999998 rpy=1.5707963267948966 1.5707963267948966 0, axis 1.2094840050743994e-31 1.0 0.0
- added joint robot_l_hip_pitch_link_l_roll_joint: type continuous, parent robot_l_hip_pitch_link, child robot_l_thigh_link, origin xyz=0.0004884400000000255 5.907999999990921e-05 0.07498434999999998 rpy=-1.5707963267949294 1.5707963267948966 0, axis -3.8518598882279653e-34 1.0 3.270422467429247e-14
- added joint robot_l_hip_yaw_link_l_pitch_joint: type continuous, parent robot_l_hip_yaw_link, child robot_l_hip_pitch_link, origin xyz=0.07499999999999987 2.877698079828406e-15 0.13629999999999995 rpy=-1.5707963267948966 2.1213866940853926e-14 1.5707963267948966, axis -2.2725973344141428e-32 2.775557561565327e-17 -1.0
- added joint robot_l_shank_link_l_ankle_joint: type continuous, parent robot_l_shank_link, child robot_l_ankle_link, origin xyz=0.0 0.3 4.440892098500626e-16 rpy=-3.141592653589792 2.241782455256438e-31 3.1554436208840472e-30, axis 1.0207428705226006e-31 -0.0 1.0
- added joint robot_l_thigh_link_l_knee_joint: type continuous, parent robot_l_thigh_link, child robot_l_shank_link, origin xyz=0.0129999999999999 0.0005000000000097771 -0.3 rpy=-1.5707963267948981 3.270422467429247e-14 -1.5707963267948966, axis -1.2210395847338845e-31 1.4849232954356037e-15 -1.0
- added joint robot_pelvis_link_l_yaw_joint: type continuous, parent robot_pelvis_link, child robot_l_hip_yaw_link, origin xyz=0.12000000000000094 0.8127999999999959 -0.1604999999999903 rpy=1.5707963267949308 2.77555756156387e-17 5.273559366969195e-16, axis -4.2755644765189156e-32 2.1213866940853923e-14 1.0
- added joint robot_pelvis_link_r_yaw_joint: type continuous, parent robot_pelvis_link, child robot_r_hip_yaw_link, origin xyz=-0.11999999999999826 0.8127999999999959 -0.1604999999999903 rpy=-1.5707963267948628 2.77555756156387e-17 5.273559366969195e-16, axis 4.2755644765189156e-32 2.1047333487160162e-14 1.0
- added joint robot_pelvis_link_torso_joint: type fixed, parent robot_pelvis_link, child robot_torso_link, origin xyz=-0.03999999999999858 0.8247999999999963 -0.2064999999999898 rpy=-1.570796326794884 2.77555756156387e-17 5.273559366969195e-16
- added joint robot_r_ankle_link_r_foot_joint: type continuous, parent robot_r_ankle_link, child robot_r_foot_link, origin xyz=0.07400000000000002 0.0 0.01 rpy=1.5707963267948966 -1.5707963267948961 0, axis -2.5037089276361443e-33 1.0 -2.105898581219543e-17
- added joint robot_r_hip_pitch_link_r_roll_joint: type continuous, parent robot_r_hip_pitch_link, child robot_r_thigh_link, origin xyz=0.0005000000000000072 0.0 0.07500000000000002 rpy=-1.5707963267948637 -1.5707963267948966 0, axis -2.1955601366083152e-32 1.0 -3.282668935420722e-14
- added joint robot_r_hip_yaw_link_r_pitch_joint: type continuous, parent robot_r_hip_yaw_link, child robot_r_hip_pitch_link, origin xyz=-0.07499999999999991 -2.877698079828406e-15 -0.13629999999999995 rpy=-1.5707963267948966 -2.1047333487160162e-14 -1.5707963267948966, axis -8.281498761229452e-33 0.0 1.0
- added joint robot_r_shank_link_r_ankle_joint: type continuous, parent robot_r_shank_link, child robot_r_ankle_link, origin xyz=0.0 -0.3 -3.552713678800501e-16 rpy=-3.1415926535897922 -1.0400021699518434e-31 0.0, axis 7.280015189638016e-32 1.5879329631222806e-30 -1.0
- added joint robot_r_thigh_link_r_knee_joint: type continuous, parent robot_r_thigh_link, child robot_r_shank_link, origin xyz=-0.013000000000000185 -0.0004999999999901661 0.3000000000000001 rpy=-1.570796326794898 3.282668935420722e-14 1.5707963267948966, axis -3.120006509880417e-32 -1.193489751472503e-15 1.0
- added joint world_to_root: type fixed, parent world, child robot_pelvis_link, origin xyz=0 0 0 rpy=1.5708 0 1.5708
