Commit message: added limits to the joints in urdf

File: simulation/isaac/assets/skeleton/skeleton_limits.urdf (robot description, URDF)
Before this commit: robot plymouth_humanoid_skeleton, 14 links, 13 joints
Links:
- link robot_l_ankle_link: geometry collision mesh filename=meshes/robot_l_ankle_link.stl scale=0.001 0.001 0.001; visual mesh filename=meshes/robot_l_ankle_link.stl scale=0.001 0.001 0.001
- link robot_l_foot_link: geometry collision mesh filename=meshes/robot_l_foot_link.stl scale=0.001 0.001 0.001; visual mesh filename=meshes/robot_l_foot_link.stl scale=0.001 0.001 0.001
- link robot_l_hip_pitch_link: geometry collision mesh filename=meshes/robot_l_hip_pitch_link.stl scale=0.001 0.001 0.001; visual mesh filename=meshes/robot_l_hip_pitch_link.stl scale=0.001 0.001 0.001
- link robot_l_hip_yaw_link: geometry collision mesh filename=meshes/robot_l_hip_yaw_link.stl scale=0.001 0.001 0.001; visual mesh filename=meshes/robot_l_hip_yaw_link.stl scale=0.001 0.001 0.001
- link robot_l_shank_link: geometry collision mesh filename=meshes/robot_l_shank_link.stl scale=0.001 0.001 0.001; visual mesh filename=meshes/robot_l_shank_link.stl scale=0.001 0.001 0.001
- link robot_l_thigh_link: geometry collision mesh filename=meshes/robot_l_thigh_link.stl scale=0.001 0.001 0.001; visual mesh filename=meshes/robot_l_thigh_link.stl scale=0.001 0.001 0.001
- link robot_pelvis_link: geometry collision mesh filename=meshes/robot_pelvis_link.stl scale=0.001 0.001 0.001; visual mesh filename=meshes/robot_pelvis_link.stl scale=0.001 0.001 0.001
- link robot_r_ankle_link: geometry collision mesh filename=meshes/robot_r_ankle_link.stl scale=0.001 0.001 0.001; visual mesh filename=meshes/robot_r_ankle_link.stl scale=0.001 0.001 0.001
- link robot_r_foot_link: geometry collision mesh filename=meshes/robot_r_foot_link.stl scale=0.001 0.001 0.001; visual mesh filename=meshes/robot_r_foot_link.stl scale=0.001 0.001 0.001
- link robot_r_hip_pitch_link: geometry collision mesh filename=meshes/robot_r_hip_pitch_link.stl scale=0.001 0.001 0.001; visual mesh filename=meshes/robot_r_hip_pitch_link.stl scale=0.001 0.001 0.001
- link robot_r_hip_yaw_link: geometry collision mesh filename=meshes/robot_r_hip_yaw_link.stl scale=0.001 0.001 0.001; visual mesh filename=meshes/robot_r_hip_yaw_link.stl scale=0.001 0.001 0.001
- link robot_r_shank_link: geometry collision mesh filename=meshes/robot_r_shank_link.stl scale=0.001 0.001 0.001; visual mesh filename=meshes/robot_r_shank_link.stl scale=0.001 0.001 0.001
- link robot_r_thigh_link: geometry collision mesh filename=meshes/robot_r_thigh_link.stl scale=0.001 0.001 0.001; visual mesh filename=meshes/robot_r_thigh_link.stl scale=0.001 0.001 0.001
- link robot_torso_link: geometry collision mesh filename=meshes/robot_torso_link.stl scale=0.001 0.001 0.001; visual mesh filename=meshes/robot_torso_link.stl scale=0.001 0.001 0.001
