Commit message: robot successfully imported into IS in correct orientation

File: simulation/isaac/assets/skeleton/skeleton.urdf (robot description, URDF)
Before this commit: robot plymouth_humanoid_skeleton, 15 links, 14 joints
Links:
- removed link world
- added link world_link
- link robot_l_ankle_link: geometry collision mesh filename=meshes/robot_l_ankle_link.stl scale=1.0 1.0 1.0; visual mesh filename=meshes/robot_l_ankle_link.stl scale=1.0 1.0 1.0
- link robot_l_foot_link: geometry collision mesh filename=meshes/robot_l_foot_link.stl scale=1.0 1.0 1.0; visual mesh filename=meshes/robot_l_foot_link.stl scale=1.0 1.0 1.0
- link robot_l_hip_pitch_link: geometry collision mesh filename=meshes/robot_l_hip_pitch_link.stl scale=1.0 1.0 1.0; visual mesh filename=meshes/robot_l_hip_pitch_link.stl scale=1.0 1.0 1.0
- link robot_l_hip_yaw_link: geometry collision mesh filename=meshes/robot_l_hip_yaw_link.stl scale=1.0 1.0 1.0; visual mesh filename=meshes/robot_l_hip_yaw_link.stl scale=1.0 1.0 1.0
- link robot_l_shank_link: geometry collision mesh filename=meshes/robot_l_shank_link.stl scale=1.0 1.0 1.0; visual mesh filename=meshes/robot_l_shank_link.stl scale=1.0 1.0 1.0
- link robot_l_thigh_link: geometry collision mesh filename=meshes/robot_l_thigh_link.stl scale=1.0 1.0 1.0; visual mesh filename=meshes/robot_l_thigh_link.stl scale=1.0 1.0 1.0
- link robot_pelvis_link: geometry collision mesh filename=meshes/robot_pelvis_link.stl scale=1.0 1.0 1.0; visual mesh filename=meshes/robot_pelvis_link.stl scale=1.0 1.0 1.0
- link robot_r_ankle_link: geometry collision mesh filename=meshes/robot_r_ankle_link.stl scale=1.0 1.0 1.0; visual mesh filename=meshes/robot_r_ankle_link.stl scale=1.0 1.0 1.0
- link robot_r_foot_link: geometry collision mesh filename=meshes/robot_r_foot_link.stl scale=1.0 1.0 1.0; visual mesh filename=meshes/robot_r_foot_link.stl scale=1.0 1.0 1.0
- link robot_r_hip_pitch_link: geometry collision mesh filename=meshes/robot_r_hip_pitch_link.stl scale=1.0 1.0 1.0; visual mesh filename=meshes/robot_r_hip_pitch_link.stl scale=1.0 1.0 1.0
- link robot_r_hip_yaw_link: geometry collision mesh filename=meshes/robot_r_hip_yaw_link.stl scale=1.0 1.0 1.0; visual mesh filename=meshes/robot_r_hip_yaw_link.stl scale=1.0 1.0 1.0
- link robot_r_shank_link: geometry collision mesh filename=meshes/robot_r_shank_link.stl scale=1.0 1.0 1.0; visual mesh filename=meshes/robot_r_shank_link.stl scale=1.0 1.0 1.0
- link robot_r_thigh_link: geometry collision mesh filename=meshes/robot_r_thigh_link.stl scale=1.0 1.0 1.0; visual mesh filename=meshes/robot_r_thigh_link.stl scale=1.0 1.0 1.0
- link robot_torso_link: geometry collision mesh filename=meshes/robot_torso_link.stl scale=1.0 1.0 1.0; visual mesh filename=meshes/robot_torso_link.stl scale=1.0 1.0 1.0
Joints:
- joint robot_l_ankle_link_l_foot_joint: axis 1.2094840050743994e-31 1.0 0.0 -> 0 1 0; origin xyz=0.07401155999999999 -5.9079999999998025e-05 0.009015649999999998 rpy=1.5707963267948966 1.5707963267948966 0 -> xyz=0.07401155999999999 -0.000059079999999998025 0.009015649999999998 rpy=1.5707963267948966 1.5707963267948966 0
- joint robot_l_hip_pitch_link_l_roll_joint: axis -3.8518598882279653e-34 1.0 3.270422467429247e-14 -> 0 1 0; origin xyz=0.0004884400000000255 5.907999999990921e-05 0.07498434999999998 rpy=-1.5707963267949294 1.5707963267948966 0 -> xyz=0.0004884400000000255 0.00005907999999990921 0.07498434999999998 rpy=-1.5707963267949294 1.5707963267948966 0
- joint robot_l_hip_yaw_link_l_pitch_joint: axis -2.2725973344141428e-32 2.775557561565327e-17 -1.0 -> 0 0 -1; origin xyz=0.07499999999999987 2.877698079828406e-15 0.13629999999999995 rpy=-1.5707963267948966 2.1213866940853926e-14 1.5707963267948966 -> xyz=0.07499999999999987 0 0.13629999999999995 rpy=-1.5707963267948966 0 1.5707963267948966
- joint robot_l_shank_link_l_ankle_joint: axis 1.0207428705226006e-31 -0.0 1.0 -> 0 0 1; origin xyz=0.0 0.3 4.440892098500626e-16 rpy=-3.141592653589792 2.241782455256438e-31 3.1554436208840472e-30 -> xyz=0 0.3 0 rpy=-3.141592653589792 0 0
- joint robot_l_thigh_link_l_knee_joint: axis -1.2210395847338845e-31 1.4849232954356037e-15 -1.0 -> 0 0 -1; origin xyz=0.0129999999999999 0.0005000000000097771 -0.3 rpy=-1.5707963267948981 3.270422467429247e-14 -1.5707963267948966 -> xyz=0.0129999999999999 0.0005000000000097771 -0.3 rpy=-1.5707963267948981 0 -1.5707963267948966
- joint robot_pelvis_link_l_yaw_joint: axis -4.2755644765189156e-32 2.1213866940853923e-14 1.0 -> 0 0 1; origin xyz=0.12000000000000094 0.8127999999999959 -0.1604999999999903 rpy=1.5707963267949308 2.77555756156387e-17 5.273559366969195e-16 -> xyz=0.12000000000000094 0.8127999999999959 -0.1604999999999903 rpy=1.5707963267949308 0 0
- joint robot_pelvis_link_r_yaw_joint: axis 4.2755644765189156e-32 2.1047333487160162e-14 1.0 -> 0 0 1; origin xyz=-0.11999999999999826 0.8127999999999959 -0.1604999999999903 rpy=-1.5707963267948628 2.77555756156387e-17 5.273559366969195e-16 -> xyz=-0.11999999999999826 0.8127999999999959 -0.1604999999999903 rpy=-1.5707963267948628 0 0
- joint robot_pelvis_link_torso_joint: origin xyz=-0.03999999999999858 0.8247999999999963 -0.2064999999999898 rpy=-1.570796326794884 2.77555756156387e-17 5.273559366969195e-16 -> xyz=-0.03999999999999858 0.8247999999999963 -0.2064999999999898 rpy=-1.570796326794884 0 0
- joint robot_r_ankle_link_r_foot_joint: axis -2.5037089276361443e-33 1.0 -2.105898581219543e-17 -> 0 1 0; origin xyz=0.07400000000000002 0.0 0.01 rpy=1.5707963267948966 -1.5707963267948961 0 -> xyz=0.07400000000000002 0 0.01 rpy=1.5707963267948966 -1.5707963267948961 0
- joint robot_r_hip_pitch_link_r_roll_joint: axis -2.1955601366083152e-32 1.0 -3.282668935420722e-14 -> 0 1 0; origin xyz=0.0005000000000000072 0.0 0.07500000000000002 rpy=-1.5707963267948637 -1.5707963267948966 0 -> xyz=0.0005000000000000072 0 0.07500000000000002 rpy=-1.5707963267948637 -1.5707963267948966 0
- joint robot_r_hip_yaw_link_r_pitch_joint: axis -8.281498761229452e-33 0.0 1.0 -> 0 0 1; origin xyz=-0.07499999999999991 -2.877698079828406e-15 -0.13629999999999995 rpy=-1.5707963267948966 -2.1047333487160162e-14 -1.5707963267948966 -> xyz=-0.07499999999999991 0 -0.13629999999999995 rpy=-1.5707963267948966 0 -1.5707963267948966
- joint robot_r_shank_link_r_ankle_joint: axis 7.280015189638016e-32 1.5879329631222806e-30 -1.0 -> 0 0 -1; origin xyz=0.0 -0.3 -3.552713678800501e-16 rpy=-3.1415926535897922 -1.0400021699518434e-31 0.0 -> xyz=0 -0.3 0 rpy=-3.1415926535897922 0 0
- joint robot_r_thigh_link_r_knee_joint: axis -3.120006509880417e-32 -1.193489751472503e-15 1.0 -> 0 0 1; origin xyz=-0.013000000000000185 -0.0004999999999901661 0.3000000000000001 rpy=-1.570796326794898 3.282668935420722e-14 1.5707963267948966 -> xyz=-0.013000000000000185 -0.0004999999999901661 0.3000000000000001 rpy=-1.570796326794898 0 1.5707963267948966
- joint world_to_root: parent world -> world_link

Commit message: Started a fresh usd file for IS with robot imported

File: simulation/isaac/assets/skeleton/skeleton.urdf (robot description, URDF)
Before this commit: robot plymouth_humanoid_skeleton, 15 links, 14 joints
Links:
- removed link world_link
Joints:
- removed joint world_to_root

Commit message: updated the joint effort and velocities at a initial values.

File: simulation/isaac/assets/skeleton/skeleton.urdf (robot description, URDF)
Before this commit: robot plymouth_humanoid_skeleton, 14 links, 13 joints
Joints:
- joint robot_l_ankle_link_l_foot_joint: limit lower=-0.261799 upper=0.261799 effort=1000000 velocity=1000000 -> lower=-0.261799 upper=0.261799 effort=45 velocity=10
- joint robot_l_hip_pitch_link_l_roll_joint: limit lower=-0.436332 upper=0.436332 effort=1000000 velocity=1000000 -> lower=-0.436332 upper=0.436332 effort=60 velocity=6
- joint robot_l_hip_yaw_link_l_pitch_joint: limit lower=-1.047198 upper=0.698132 effort=1000000 velocity=1000000 -> lower=-1.047198 upper=0.698132 effort=60 velocity=6
- joint robot_l_shank_link_l_ankle_joint: limit lower=-0.610865 upper=0.436332 effort=1000000 velocity=1000000 -> lower=-0.610865 upper=0.436332 effort=45 velocity=10
- joint robot_l_thigh_link_l_knee_joint: limit lower=-2.094395 upper=0.0 effort=1000000 velocity=1000000 -> lower=-2.094395 upper=0.0 effort=90 velocity=8
- joint robot_pelvis_link_l_yaw_joint: limit lower=-0.523599 upper=0.523599 effort=1000000 velocity=1000000 -> lower=-0.523599 upper=0.523599 effort=60 velocity=6
- joint robot_pelvis_link_r_yaw_joint: limit lower=-0.523599 upper=0.523599 effort=1000000 velocity=1000000 -> lower=-0.523599 upper=0.523599 effort=60 velocity=6
- joint robot_r_ankle_link_r_foot_joint: limit lower=-0.261799 upper=0.261799 effort=1000000 velocity=1000000 -> lower=-0.261799 upper=0.261799 effort=45 velocity=10
- joint robot_r_hip_pitch_link_r_roll_joint: limit lower=-0.436332 upper=0.436332 effort=1000000 velocity=1000000 -> lower=-0.436332 upper=0.436332 effort=60 velocity=6
- joint robot_r_hip_yaw_link_r_pitch_joint: limit lower=-1.047198 upper=0.698132 effort=1000000 velocity=1000000 -> lower=-1.047198 upper=0.698132 effort=60 velocity=6
- joint robot_r_shank_link_r_ankle_joint: limit lower=-0.610865 upper=0.436332 effort=1000000 velocity=1000000 -> lower=-0.610865 upper=0.436332 effort=45 velocity=10
- joint robot_r_thigh_link_r_knee_joint: limit lower=-2.094395 upper=0.0 effort=1000000 velocity=1000000 -> lower=-2.094395 upper=0.0 effort=90 velocity=8

Commit message: added a urdf cleaner and ran it
This removed all the values which use the scientific notation, changing those affected values with 0 instead if below a threshold. This was to ensure the urdf file would run in IS/IL

File: simulation/isaac/assets/skeleton/skeleton.urdf (robot description, URDF)
Before this commit: robot export_v2, 14 links, 13 joints
Joints:
- joint robot_l_ankle_link_l_foot_joint: axis 1.2094840050743994e-31 1.0 0.0 -> 0 1.0 0
- joint robot_l_hip_pitch_link_l_roll_joint: axis -3.8518598882279653e-34 1.0 3.270422467429247e-14 -> 0 1.0 0
- joint robot_l_hip_yaw_link_l_pitch_joint: axis -2.2725973344141428e-32 2.775557561565327e-17 -1.0 -> 0 0 -1.0; origin xyz=0.07499999999999987 2.877698079828406e-15 0.13629999999999995 rpy=-1.5707963267948966 2.1213866940853926e-14 1.5707963267948966 -> xyz=0.07499999999999987 0 0.13629999999999995 rpy=-1.5707963267948966 0 1.5707963267948966
- joint robot_l_shank_link_l_ankle_joint: axis 1.0207428705226006e-31 -0.0 1.0 -> 0 0 1.0; origin xyz=0.0 0.3 4.440892098500626e-16 rpy=-3.141592653589792 2.241782455256438e-31 3.1554436208840472e-30 -> xyz=0 0.3 0 rpy=-3.141592653589792 0 0
- joint robot_l_thigh_link_l_knee_joint: axis -1.2210395847338845e-31 1.4849232954356037e-15 -1.0 -> 0 0 -1.0; origin xyz=0.0129999999999999 0.0005000000000097771 -0.3 rpy=-1.5707963267948981 3.270422467429247e-14 -1.5707963267948966 -> xyz=0.0129999999999999 0.0005000000000097771 -0.3 rpy=-1.5707963267948981 0 -1.5707963267948966
- joint robot_pelvis_link_l_yaw_joint: axis -4.2755644765189156e-32 2.1213866940853923e-14 1.0 -> 0 0 1.0; origin xyz=0.12000000000000094 0.8127999999999959 -0.1604999999999903 rpy=1.5707963267949308 2.77555756156387e-17 5.273559366969195e-16 -> xyz=0.12000000000000094 0.8127999999999959 -0.1604999999999903 rpy=1.5707963267949308 0 0
- joint robot_pelvis_link_r_yaw_joint: axis 4.2755644765189156e-32 2.1047333487160162e-14 1.0 -> 0 0 1.0; origin xyz=-0.11999999999999826 0.8127999999999959 -0.1604999999999903 rpy=-1.5707963267948628 2.77555756156387e-17 5.273559366969195e-16 -> xyz=-0.11999999999999826 0.8127999999999959 -0.1604999999999903 rpy=-1.5707963267948628 0 0
- joint robot_pelvis_link_torso_joint: origin xyz=-0.03999999999999858 0.8247999999999963 -0.2064999999999898 rpy=-1.570796326794884 2.77555756156387e-17 5.273559366969195e-16 -> xyz=-0.03999999999999858 0.8247999999999963 -0.2064999999999898 rpy=-1.570796326794884 0 0
- joint robot_r_ankle_link_r_foot_joint: axis -2.5037089276361443e-33 1.0 -2.105898581219543e-17 -> 0 1.0 0; origin xyz=0.07400000000000002 0.0 0.01 rpy=1.5707963267948966 -1.5707963267948961 0 -> xyz=0.07400000000000002 0 0.01 rpy=1.5707963267948966 -1.5707963267948961 0
- joint robot_r_hip_pitch_link_r_roll_joint: axis -2.1955601366083152e-32 1.0 -3.282668935420722e-14 -> 0 1.0 0; origin xyz=0.0005000000000000072 0.0 0.07500000000000002 rpy=-1.5707963267948637 -1.5707963267948966 0 -> xyz=0.0005000000000000072 0 0.07500000000000002 rpy=-1.5707963267948637 -1.5707963267948966 0
- joint robot_r_hip_yaw_link_r_pitch_joint: axis -8.281498761229452e-33 0.0 1.0 -> 0 0 1.0; origin xyz=-0.07499999999999991 -2.877698079828406e-15 -0.13629999999999995 rpy=-1.5707963267948966 -2.1047333487160162e-14 -1.5707963267948966 -> xyz=-0.07499999999999991 0 -0.13629999999999995 rpy=-1.5707963267948966 0 -1.5707963267948966
- joint robot_r_shank_link_r_ankle_joint: axis 7.280015189638016e-32 1.5879329631222806e-30 -1.0 -> 0 0 -1.0; origin xyz=0.0 -0.3 -3.552713678800501e-16 rpy=-3.1415926535897922 -1.0400021699518434e-31 0.0 -> xyz=0 -0.3 0 rpy=-3.1415926535897922 0 0
- joint robot_r_thigh_link_r_knee_joint: axis -3.120006509880417e-32 -1.193489751472503e-15 1.0 -> 0 0 1.0; origin xyz=-0.013000000000000185 -0.0004999999999901661 0.3000000000000001 rpy=-1.570796326794898 3.282668935420722e-14 1.5707963267948966 -> xyz=-0.013000000000000185 -0.0004999999999901661 0.3000000000000001 rpy=-1.570796326794898 0 1.5707963267948966

Commit message: fixed the orientation issue from the urdf file

File: simulation/isaac/assets/skeleton/skeleton.urdf (robot description, URDF)
Before this commit: robot Robot, 14 links, 13 joints
Links:
- added link isaac_zup_root
Joints:
- added joint isaac_zup_root_joint: type fixed, parent isaac_zup_root, child robot_pelvis_link, origin xyz=0 0 0 rpy=1.57079632679 0 0

Commit message: Fixed the URDF to rotate the robot 180 degrees around the Z axis as it was trying to walk backward in training.

File: simulation/isaac/assets/skeleton/skeleton.urdf (robot description, URDF)
Before this commit: robot Robot, 15 links, 14 joints
Joints:
- joint isaac_zup_root_joint: origin xyz=0 0 0 rpy=1.57079632679 0 0 -> xyz=0 0 0 rpy=1.57079632679 0 3.14159265359

Commit message: Updated the USD to correct the robot facing in the wrong direction

File: simulation/isaac/assets/skeleton/skeleton.urdf (robot description, URDF)
Before this commit: robot Robot, 15 links, 14 joints
Joints:
- joint isaac_zup_root_joint: origin xyz=0 0 0 rpy=1.57079632679 0 3.14159265359 -> xyz=0 0 0 rpy=1.57079632679 0 1.57079632679

Commit message: Exported URDF again and created new USD

File: simulation/isaac/assets/skeleton/skeleton.urdf (robot description, URDF)
Before this commit: robot Robot, 15 links, 14 joints
Joints:
- joint robot_l_ankle_link_l_foot_joint: limit lower=-0.261799 upper=0.261799 effort=45 velocity=10 -> lower=-0.261799 upper=0.261799 effort=1000000 velocity=1000000
- joint robot_l_hip_pitch_link_l_roll_joint: limit lower=-0.436332 upper=0.436332 effort=60 velocity=6 -> lower=-0.436332 upper=0.436332 effort=1000000 velocity=1000000; origin xyz=0.0004884400000000255 5.907999999990921e-05 0.07498434999999998 rpy=-1.5707963267949294 1.5707963267948966 0 -> xyz=0.00048843999999999 -5.907999999990921e-05 -0.07498434999999999 rpy=-1.5707963267948966 -1.5707963267948966 0
- joint robot_l_hip_yaw_link_l_pitch_joint: limit lower=-1.047198 upper=0.698132 effort=60 velocity=6 -> lower=-0.698132 upper=1.047198 effort=1000000 velocity=1000000; origin xyz=0.07499999999999987 0 0.13629999999999995 rpy=-1.5707963267948966 0 1.5707963267948966 -> xyz=0.07499999999999998 0 0.13629999999999995 rpy=1.5707963267948966 0 1.5707963267948966
- joint robot_l_shank_link_l_ankle_joint: limit lower=-0.610865 upper=0.436332 effort=45 velocity=10 -> lower=-0.610865 upper=0.610865 effort=1000000 velocity=1000000; origin xyz=0 0.3 0 rpy=-3.141592653589792 0 0 -> xyz=0 -0.3 0 rpy=0 0 0
- joint robot_l_thigh_link_l_knee_joint: limit lower=-2.094395 upper=0.0 effort=90 velocity=8 -> lower=0.0 upper=2.094395 effort=1000000 velocity=1000000; origin xyz=0.0129999999999999 0.0005000000000097771 -0.3 rpy=-1.5707963267948981 0 -1.5707963267948966 -> xyz=0.013000000000000008 -0.0004999999999999716 0.3 rpy=-1.5707963267948966 0 1.5707963267948966
- joint robot_pelvis_link_l_yaw_joint: limit lower=-0.523599 upper=0.523599 effort=60 velocity=6 -> lower=-0.523599 upper=0.523599 effort=1000000 velocity=1000000; origin xyz=0.12000000000000094 0.8127999999999959 -0.1604999999999903 rpy=1.5707963267949308 0 0 -> xyz=0.12000000000000094 0.8127999999999959 -0.1604999999999903 rpy=1.5707963267949094 0 0
- joint robot_pelvis_link_r_yaw_joint: axis 0 0 1.0 -> 0 0 -1.0; limit lower=-0.523599 upper=0.523599 effort=60 velocity=6 -> lower=-0.523599 upper=0.523599 effort=1000000 velocity=1000000; origin xyz=-0.11999999999999826 0.8127999999999959 -0.1604999999999903 rpy=-1.5707963267948628 0 0 -> xyz=-0.11999999999999826 0.8127999999999959 -0.1604999999999903 rpy=1.5707963267949094 0 0
- joint robot_r_ankle_link_r_foot_joint: axis 0 1.0 0 -> 0 -1.0 0; limit lower=-0.261799 upper=0.261799 effort=45 velocity=10 -> lower=-0.261799 upper=0.261799 effort=1000000 velocity=1000000; origin xyz=0.07400000000000002 0 0.01 rpy=1.5707963267948966 -1.5707963267948961 0 -> xyz=0.07400000000000001 0 -0.01 rpy=1.5707963267948966 1.5707963267948966 0
- joint robot_r_hip_pitch_link_r_roll_joint: axis 0 1.0 0 -> 0 -1.0 0; limit lower=-0.436332 upper=0.436332 effort=60 velocity=6 -> lower=-0.436332 upper=0.436332 effort=1000000 velocity=1000000; origin xyz=0.0005000000000000072 0 0.07500000000000002 rpy=-1.5707963267948637 -1.5707963267948966 0 -> xyz=0.0005000000000000072 0 0.07500000000000002 rpy=-1.5707963267948966 -1.5707963267948966 0
- joint robot_r_hip_yaw_link_r_pitch_joint: axis 0 0 1.0 -> 0 0 -1.0; limit lower=-1.047198 upper=0.698132 effort=60 velocity=6 -> lower=-0.698132 upper=1.047198 effort=1000000 velocity=1000000; origin xyz=-0.07499999999999991 0 -0.13629999999999995 rpy=-1.5707963267948966 0 -1.5707963267948966 -> xyz=-0.07500000000000002 0 0.13629999999999995 rpy=1.5707963267948966 0 1.5707963267948966
- joint robot_r_shank_link_r_ankle_joint: axis 0 0 -1.0 -> 0 0 1.0; limit lower=-0.610865 upper=0.436332 effort=45 velocity=10 -> lower=-0.610865 upper=0.610865 effort=1000000 velocity=1000000; origin xyz=0 -0.3 0 rpy=-3.1415926535897922 0 0 -> xyz=0 -0.3 0 rpy=0 0 0
- joint robot_r_thigh_link_r_knee_joint: axis 0 0 1.0 -> 0 0 -1.0; limit lower=-2.094395 upper=0.0 effort=90 velocity=8 -> lower=0.0 upper=2.094395 effort=1000000 velocity=1000000; origin xyz=-0.013000000000000185 -0.0004999999999901661 0.3000000000000001 rpy=-1.570796326794898 0 1.5707963267948966 -> xyz=-0.013000000000000008 -0.0005000000000000072 0.3000000000000001 rpy=-1.5707963267948966 0 1.5707963267948966

Commit message: Corrected the right foot on the robot and remade the usd file.

File: simulation/isaac/assets/skeleton/skeleton.urdf (robot description, URDF)
Before this commit: robot Robot, 15 links, 14 joints
Joints:
- joint robot_l_hip_pitch_link_l_roll_joint: origin xyz=0.00048843999999999 -5.907999999990921e-05 -0.07498434999999999 rpy=-1.5707963267948966 -1.5707963267948966 0 -> xyz=0.00048843999999999 -5.907999999990921e-05 -0.07498435 rpy=-1.5707963267948966 -1.5707963267948966 0
- joint robot_l_hip_yaw_link_l_pitch_joint: origin xyz=0.07499999999999998 0 0.13629999999999995 rpy=1.5707963267948966 0 1.5707963267948966 -> xyz=0.075 0 0.13629999999999995 rpy=1.5707963267948966 0 1.5707963267948966
- joint robot_pelvis_link_l_yaw_joint: origin xyz=0.12000000000000094 0.8127999999999959 -0.1604999999999903 rpy=1.5707963267949094 0 0 -> xyz=0.12000000000000183 0.8127999999999906 -0.16050000405310783 rpy=1.5707963267949094 0 0
- joint robot_pelvis_link_r_yaw_joint: origin xyz=-0.11999999999999826 0.8127999999999959 -0.1604999999999903 rpy=1.5707963267949094 0 0 -> xyz=-0.11999999999999739 0.8127999999999906 -0.1605000040531078 rpy=1.5707963267949094 0 0
- joint robot_pelvis_link_torso_joint: origin xyz=-0.03999999999999858 0.8247999999999963 -0.2064999999999898 rpy=-1.570796326794884 0 0 -> xyz=-0.03999999999999768 0.8247999999999912 -0.2065000040531073 rpy=-1.5707963267948837 0 0
- joint robot_r_ankle_link_r_foot_joint: origin xyz=0.07400000000000001 0 -0.01 rpy=1.5707963267948966 1.5707963267948966 0 -> xyz=0.07400000000000001 0 -0.009000000000000005 rpy=1.5707963267948966 1.5707963267948966 0
- joint robot_r_hip_pitch_link_r_roll_joint: origin xyz=0.0005000000000000072 0 0.07500000000000002 rpy=-1.5707963267948966 -1.5707963267948966 0 -> xyz=0.0005000000000000072 0 0.075 rpy=-1.5707963267948966 -1.5707963267948966 0
- joint robot_r_hip_yaw_link_r_pitch_joint: origin xyz=-0.07500000000000002 0 0.13629999999999995 rpy=1.5707963267948966 0 1.5707963267948966 -> xyz=-0.075 0 0.13629999999999995 rpy=1.5707963267948966 0 1.5707963267948966
