Commit message: Update robot.urdf
Cleaned up the urdf file

File: simulation/isaac/assets/robot/robot.urdf (robot description, URDF)
Before this commit: robot robot, 16 links, 15 joints
Joints:
- joint l_ankle_link_l_foot_joint: axis 1.0 0.0 -2.16107724819376e-16 -> 1.0 0 0; origin xyz=0.07402717 0.009000000000000005 3.743000000000052e-05 rpy=-6.4254155418928814e-15 -0.0 0.0 -> xyz=0.07402717 0.009000000000000005 3.743000000000052e-05 rpy=0 0 0
- joint l_hip_pitch_link_l_roll_joint: axis 1.0 0.0 -2.220446049246316e-16 -> 1.0 0 0; origin xyz=0.0 0.075 0.0012999999999999908 rpy=-1.5707963267948966 -1.5707963267948963 0 -> xyz=0 0.075 0.0012999999999999908 rpy=-1.5707963267948966 -1.5707963267948963 0
- joint l_hip_yaw_link_l_pitch_joint: axis 0.0 1.0 -1.222700479015263e-16 -> 0 1.0 0; origin xyz=-1.1048011099959547e-16 -0.07499999999999755 0.13630000000000136 rpy=1.2227004790152155e-16 1.5707963267948786 0 -> xyz=0 -0.07499999999999755 0.13630000000000136 rpy=0 1.5707963267948786 0
- joint l_shank_link_l_ankle_joint: axis -0.0 1.0 2.465190328815662e-32 -> 0 1.0 0; origin xyz=0.0 -0.3 -3.552713678800501e-17 rpy=1.5707963267948968 -0.0 0.0 -> xyz=0 -0.3 0 rpy=1.5707963267948968 0 0
- joint l_thigh_link_l_knee_joint: axis 0.0 1.2246467991536624e-16 -1.0 -> 0 0 -1.0; origin xyz=0.003499999999999997 -0.3 -0.013000000000000008 rpy=-1.2246467991481818e-16 -0.0 0.0 -> xyz=0.003499999999999997 -0.3 -0.013000000000000008 rpy=0 0 0
- joint pelvis_link_l_yaw_joint: axis 0.0 1.7918659470244052e-14 1.0 -> 0 0 1.0; origin xyz=0.11999999999233989 3.066148575681922e-12 -0.012 rpy=-3.1415926535897754 -0.0 -1.570796326794897 -> xyz=0.11999999999233989 3.066148575681922e-12 -0.012 rpy=-3.1415926535897754 0 -1.570796326794897
- joint pelvis_link_r_yaw_joint: axis 0.0 -1.7918659470244052e-14 -1.0 -> 0 0 -1.0; origin xyz=-0.12000000000765933 3.0662609857631655e-12 -0.012 rpy=-3.1415926535897754 -0.0 -1.570796326794897 -> xyz=-0.12000000000765933 3.0662609857631655e-12 -0.012 rpy=-3.1415926535897754 0 -1.570796326794897
- joint pelvis_link_torso_joint: origin xyz=-7.659717486428201e-12 -0.0004999999969337935 0.015 rpy=-2.775557561562882e-16 -0.0 -1.570796326794897 -> xyz=-7.659717486428201e-12 -0.0004999999969337935 0.015 rpy=0 0 -1.570796326794897
- joint r_ankle_link_r_foot_joint: axis -1.0 0.0 2.16107724819376e-16 -> -1.0 0 0; origin xyz=0.07397279 0.009000000000000005 3.7410000000051014e-05 rpy=6.4254155418928814e-15 -0.0 0.0 -> xyz=0.07397279 0.009000000000000005 3.7410000000051014e-05 rpy=0 0 0
- joint r_hip_pitch_link_r_roll_joint: axis -1.0 0.0 2.220446049251407e-16 -> -1.0 0 0; origin xyz=0.0 -0.075 0.0013000000000000093 rpy=-1.5707963267948966 -1.5707963267948963 0 -> xyz=0 -0.075 0.0013000000000000093 rpy=-1.5707963267948966 -1.5707963267948963 0
- joint r_hip_yaw_link_r_pitch_joint: axis 0.0 1.0 -1.222700479015263e-16 -> 0 1.0 0; origin xyz=-1.1048011099959325e-16 0.07500000000000245 0.13629999999999867 rpy=1.2227004790152155e-16 1.5707963267948786 0 -> xyz=0 0.07500000000000245 0.13629999999999867 rpy=0 1.5707963267948786 0
- joint r_shank_link_r_ankle_joint: axis 0.0 -1.0 2.465190328815662e-32 -> 0 -1.0 0; origin xyz=0.0 -0.3 0.0 rpy=-1.5707963267948966 -0.0 0.0 -> xyz=0 -0.3 0 rpy=-1.5707963267948966 0 0
- joint r_thigh_link_r_knee_joint: axis 0.0 6.308915089505042e-28 -1.0 -> 0 0 -1.0; origin xyz=0.0035000000000000027 -0.3 0.013000000000000008 rpy=-8.689919168591649e-28 -0.0 0.0 -> xyz=0.0035000000000000027 -0.3 0.013000000000000008 rpy=0 0 0
- joint torso_link_imu_joint: origin xyz=-0.008200000000000002 0.03699099999999994 0.22879999 rpy=-1.5751289161869385e-15 -1.5707963267948963 0 -> xyz=-0.008200000000000002 0.03699099999999994 0.22879999 rpy=0 -1.5707963267948963 0

Commit message: Updated the robot again after changing the unit in fusion360

File: simulation/isaac/assets/robot/robot.urdf (robot description, URDF)
Before this commit: robot robot, 16 links, 15 joints
Links:
- removed link ori_correction
Joints:
- removed joint ori_correction

Commit message: Update robot.urdf
Added the oritention rotation correction

File: simulation/isaac/assets/robot/robot.urdf (robot description, URDF)
Before this commit: robot robot, 15 links, 14 joints
Links:
- added link ori_correct
Joints:
- added joint ori_correct: type fixed, parent ori_correct, child pelvis_link, origin xyz=0 0 0 rpy=0 0 1.57079632679

Commit message: added a pelvis height transform to make sure the feet are above ground, then made usd

File: simulation/isaac/assets/robot/robot.urdf (robot description, URDF)
Before this commit: robot robot, 16 links, 15 joints
Joints:
- joint ori_correct: origin xyz=0 0 0 rpy=0 0 1.57079632679 -> xyz=0 0 0.84 rpy=0 0 1.57079632679

Commit message: Update robot.urdf
changed the name of link

File: simulation/isaac/assets/robot/robot.urdf (robot description, URDF)
Before this commit: robot robot, 16 links, 15 joints
Links:
- removed link ori_correct
- added link root
Joints:
- removed joint ori_correct
- added joint root: type fixed, parent root, child pelvis_link, origin xyz=0 0 0.84 rpy=0 0 1.57079632679

Commit message: cleaned urdf for final robot

File: simulation/isaac/assets/robot/robot.urdf (robot description, URDF)
Before this commit: robot robot, 16 links, 15 joints
Links:
- removed link root
- link torso_link: mass 11.977159824591427 -> 11.97706793583374
Joints:
- removed joint pelvis_link_torso_joint
- removed joint root
- added joint torso_link_torso_joint: type fixed, parent torso_link, child pelvis_link, origin xyz=-0.2500000019149655 -0.0009000000000000097 0.08679999999684095 rpy=0 -1.5707963267948963 0
- joint pelvis_link_l_yaw_joint: origin xyz=0.11999999999233989 3.066148575681922e-12 -0.012 rpy=-3.1415926535897754 0 -1.570796326794897 -> xyz=-0.0005 -0.027000000000000003 -0.12 rpy=1.5707963267949145 0 0
- joint pelvis_link_r_yaw_joint: origin xyz=-0.12000000000765933 3.0662609857631655e-12 -0.012 rpy=-3.1415926535897754 0 -1.570796326794897 -> xyz=-0.0005 -0.027000000000000003 0.12 rpy=1.5707963267949145 0 0
- joint torso_link_imu_joint: origin xyz=-0.008200000000000002 0.03699099999999994 0.22879999 rpy=0 -1.5707963267948963 0 -> xyz=-0.21300900191496547 0.22789999000000002 0.05299999999684098 rpy=3.1415926535897913 0 1.5707963267948963

Commit message: Revert "cleaned urdf for final robot"
This reverts commit 2198c4d3521ca9078436860fbb202f5907892b46.

File: simulation/isaac/assets/robot/robot.urdf (robot description, URDF)
Before this commit: robot robot_final, 15 links, 14 joints
Links:
- added link root
- link torso_link: mass 11.97706793583374 -> 11.977159824591427
Joints:
- removed joint torso_link_torso_joint
- added joint pelvis_link_torso_joint: type fixed, parent pelvis_link, child torso_link, origin xyz=-7.659717486428201e-12 -0.0004999999969337935 0.015 rpy=0 0 -1.570796326794897
- added joint root: type fixed, parent root, child pelvis_link, origin xyz=0 0 0.84 rpy=0 0 1.57079632679
- joint pelvis_link_l_yaw_joint: origin xyz=-0.0005 -0.027000000000000003 -0.12 rpy=1.5707963267949145 0 0 -> xyz=0.11999999999233989 3.066148575681922e-12 -0.012 rpy=-3.1415926535897754 0 -1.570796326794897
- joint pelvis_link_r_yaw_joint: origin xyz=-0.0005 -0.027000000000000003 0.12 rpy=1.5707963267949145 0 0 -> xyz=-0.12000000000765933 3.0662609857631655e-12 -0.012 rpy=-3.1415926535897754 0 -1.570796326794897
- joint torso_link_imu_joint: origin xyz=-0.21300900191496547 0.22789999000000002 0.05299999999684098 rpy=3.1415926535897913 0 1.5707963267948963 -> xyz=-0.008200000000000002 0.03699099999999994 0.22879999 rpy=0 -1.5707963267948963 0

Commit message: Updated the urdf

File: simulation/isaac/assets/robot/robot.urdf (robot description, URDF)
Before this commit: robot robot, 16 links, 15 joints
Links:
- link torso_link: mass 11.977159824591427 -> 11.97706793583374
Joints:
- removed joint pelvis_link_torso_joint
- added joint torso_link_torso_joint: type fixed, parent torso_link, child pelvis_link, origin xyz=-0.2500000019149655 -0.0009000000000000097 0.08679999999684095 rpy=-2.151057110211245e-16 -1.5707963267948963 0
- joint l_ankle_link_l_foot_joint: axis 1.0 0 0 -> 1.0 0.0 -2.16107724819376e-16; origin xyz=0.07402717 0.009000000000000005 3.743000000000052e-05 rpy=0 0 0 -> xyz=0.07402717 0.009000000000000005 3.743000000000052e-05 rpy=-6.4254155418928814e-15 -0.0 0.0
- joint l_hip_pitch_link_l_roll_joint: axis 1.0 0 0 -> 1.0 0.0 -2.220446049246316e-16; origin xyz=0 0.075 0.0012999999999999908 rpy=-1.5707963267948966 -1.5707963267948963 0 -> xyz=0.0 0.075 0.0012999999999999908 rpy=-1.5707963267948966 -1.5707963267948963 0
- joint l_hip_yaw_link_l_pitch_joint: axis 0 1.0 0 -> 0.0 1.0 -1.222700479015263e-16; origin xyz=0 -0.07499999999999755 0.13630000000000136 rpy=0 1.5707963267948786 0 -> xyz=-1.1048011099959547e-16 -0.07499999999999755 0.13630000000000136 rpy=1.2227004790152155e-16 1.5707963267948786 0
- joint l_shank_link_l_ankle_joint: axis 0 1.0 0 -> -0.0 1.0 2.465190328815662e-32; origin xyz=0 -0.3 0 rpy=1.5707963267948968 0 0 -> xyz=0.0 -0.3 -3.552713678800501e-17 rpy=1.5707963267948968 -0.0 0.0
- joint l_thigh_link_l_knee_joint: axis 0 0 -1.0 -> 0.0 1.2246467991536624e-16 -1.0; origin xyz=0.003499999999999997 -0.3 -0.013000000000000008 rpy=0 0 0 -> xyz=0.003499999999999997 -0.3 -0.013000000000000008 rpy=-1.2246467991481818e-16 -0.0 0.0
- joint pelvis_link_l_yaw_joint: axis 0 0 1.0 -> 0.0 1.7918659470244052e-14 1.0; origin xyz=0.11999999999233989 3.066148575681922e-12 -0.012 rpy=-3.1415926535897754 0 -1.570796326794897 -> xyz=-0.0005 -0.027000000000000003 -0.12 rpy=1.5707963267949145 -0.0 0.0
- joint pelvis_link_r_yaw_joint: axis 0 0 -1.0 -> 0.0 -1.7918659470244052e-14 -1.0; origin xyz=-0.12000000000765933 3.0662609857631655e-12 -0.012 rpy=-3.1415926535897754 0 -1.570796326794897 -> xyz=-0.0005 -0.027000000000000003 0.12 rpy=1.5707963267949145 -0.0 0.0
- joint r_ankle_link_r_foot_joint: axis -1.0 0 0 -> -1.0 0.0 2.16107724819376e-16; origin xyz=0.07397279 0.009000000000000005 3.7410000000051014e-05 rpy=0 0 0 -> xyz=0.07397279 0.009000000000000005 3.7410000000051014e-05 rpy=6.4254155418928814e-15 -0.0 0.0
- joint r_hip_pitch_link_r_roll_joint: axis -1.0 0 0 -> -1.0 0.0 2.220446049251407e-16; origin xyz=0 -0.075 0.0013000000000000093 rpy=-1.5707963267948966 -1.5707963267948963 0 -> xyz=0.0 -0.075 0.0013000000000000093 rpy=-1.5707963267948966 -1.5707963267948963 0
- joint r_hip_yaw_link_r_pitch_joint: axis 0 1.0 0 -> 0.0 1.0 -1.222700479015263e-16; origin xyz=0 0.07500000000000245 0.13629999999999867 rpy=0 1.5707963267948786 0 -> xyz=-1.1048011099959325e-16 0.07500000000000245 0.13629999999999867 rpy=1.2227004790152155e-16 1.5707963267948786 0
- joint r_shank_link_r_ankle_joint: axis 0 -1.0 0 -> 0.0 -1.0 2.465190328815662e-32; origin xyz=0 -0.3 0 rpy=-1.5707963267948966 0 0 -> xyz=0.0 -0.3 0.0 rpy=-1.5707963267948966 -0.0 0.0
- joint r_thigh_link_r_knee_joint: axis 0 0 -1.0 -> 0.0 6.308915089505042e-28 -1.0; origin xyz=0.0035000000000000027 -0.3 0.013000000000000008 rpy=0 0 0 -> xyz=0.0035000000000000027 -0.3 0.013000000000000008 rpy=-8.689919168591649e-28 -0.0 0.0
- joint torso_link_imu_joint: origin xyz=-0.008200000000000002 0.03699099999999994 0.22879999 rpy=0 -1.5707963267948963 0 -> xyz=-0.21300900191496547 0.22789999000000002 0.05299999999684098 rpy=3.1415926535897913 2.775557561562813e-17 1.5707963267948963

Commit message: Update robot.urdf
cleaner

File: simulation/isaac/assets/robot/robot.urdf (robot description, URDF)
Before this commit: robot robot, 16 links, 15 joints
Joints:
- joint l_ankle_link_l_foot_joint: axis 1.0 0.0 -2.16107724819376e-16 -> 1.0 0 0; origin xyz=0.07402717 0.009000000000000005 3.743000000000052e-05 rpy=-6.4254155418928814e-15 -0.0 0.0 -> xyz=0.07402717 0.009000000000000005 3.743000000000052e-05 rpy=0 0 0
- joint l_hip_pitch_link_l_roll_joint: axis 1.0 0.0 -2.220446049246316e-16 -> 1.0 0 0; origin xyz=0.0 0.075 0.0012999999999999908 rpy=-1.5707963267948966 -1.5707963267948963 0 -> xyz=0 0.075 0.0012999999999999908 rpy=-1.5707963267948966 -1.5707963267948963 0
- joint l_hip_yaw_link_l_pitch_joint: axis 0.0 1.0 -1.222700479015263e-16 -> 0 1.0 0; origin xyz=-1.1048011099959547e-16 -0.07499999999999755 0.13630000000000136 rpy=1.2227004790152155e-16 1.5707963267948786 0 -> xyz=0 -0.07499999999999755 0.13630000000000136 rpy=0 1.5707963267948786 0
- joint l_shank_link_l_ankle_joint: axis -0.0 1.0 2.465190328815662e-32 -> 0 1.0 0; origin xyz=0.0 -0.3 -3.552713678800501e-17 rpy=1.5707963267948968 -0.0 0.0 -> xyz=0 -0.3 0 rpy=1.5707963267948968 0 0
- joint l_thigh_link_l_knee_joint: axis 0.0 1.2246467991536624e-16 -1.0 -> 0 0 -1.0; origin xyz=0.003499999999999997 -0.3 -0.013000000000000008 rpy=-1.2246467991481818e-16 -0.0 0.0 -> xyz=0.003499999999999997 -0.3 -0.013000000000000008 rpy=0 0 0
- joint pelvis_link_l_yaw_joint: axis 0.0 1.7918659470244052e-14 1.0 -> 0 0 1.0; origin xyz=-0.0005 -0.027000000000000003 -0.12 rpy=1.5707963267949145 -0.0 0.0 -> xyz=-0.0005 -0.027000000000000003 -0.12 rpy=1.5707963267949145 0 0
- joint pelvis_link_r_yaw_joint: axis 0.0 -1.7918659470244052e-14 -1.0 -> 0 0 -1.0; origin xyz=-0.0005 -0.027000000000000003 0.12 rpy=1.5707963267949145 -0.0 0.0 -> xyz=-0.0005 -0.027000000000000003 0.12 rpy=1.5707963267949145 0 0
- joint r_ankle_link_r_foot_joint: axis -1.0 0.0 2.16107724819376e-16 -> -1.0 0 0; origin xyz=0.07397279 0.009000000000000005 3.7410000000051014e-05 rpy=6.4254155418928814e-15 -0.0 0.0 -> xyz=0.07397279 0.009000000000000005 3.7410000000051014e-05 rpy=0 0 0
- joint r_hip_pitch_link_r_roll_joint: axis -1.0 0.0 2.220446049251407e-16 -> -1.0 0 0; origin xyz=0.0 -0.075 0.0013000000000000093 rpy=-1.5707963267948966 -1.5707963267948963 0 -> xyz=0 -0.075 0.0013000000000000093 rpy=-1.5707963267948966 -1.5707963267948963 0
- joint r_hip_yaw_link_r_pitch_joint: axis 0.0 1.0 -1.222700479015263e-16 -> 0 1.0 0; origin xyz=-1.1048011099959325e-16 0.07500000000000245 0.13629999999999867 rpy=1.2227004790152155e-16 1.5707963267948786 0 -> xyz=0 0.07500000000000245 0.13629999999999867 rpy=0 1.5707963267948786 0
- joint r_shank_link_r_ankle_joint: axis 0.0 -1.0 2.465190328815662e-32 -> 0 -1.0 0; origin xyz=0.0 -0.3 0.0 rpy=-1.5707963267948966 -0.0 0.0 -> xyz=0 -0.3 0 rpy=-1.5707963267948966 0 0
- joint r_thigh_link_r_knee_joint: axis 0.0 6.308915089505042e-28 -1.0 -> 0 0 -1.0; origin xyz=0.0035000000000000027 -0.3 0.013000000000000008 rpy=-8.689919168591649e-28 -0.0 0.0 -> xyz=0.0035000000000000027 -0.3 0.013000000000000008 rpy=0 0 0
- joint torso_link_imu_joint: origin xyz=-0.21300900191496547 0.22789999000000002 0.05299999999684098 rpy=3.1415926535897913 2.775557561562813e-17 1.5707963267948963 -> xyz=-0.21300900191496547 0.22789999000000002 0.05299999999684098 rpy=3.1415926535897913 0 1.5707963267948963
- joint torso_link_torso_joint: origin xyz=-0.2500000019149655 -0.0009000000000000097 0.08679999999684095 rpy=-2.151057110211245e-16 -1.5707963267948963 0 -> xyz=-0.2500000019149655 -0.0009000000000000097 0.08679999999684095 rpy=0 -1.5707963267948963 0

Commit message: URDF clean

File: simulation/isaac/assets/robot/robot.urdf (robot description, URDF)
Before this commit: robot robot, 16 links, 15 joints
Joints:
- joint l_ankle_link_l_foot_joint: axis 1.0 0.0 -2.16107724819376e-16 -> 1.0 0 0; origin xyz=0.07402717 0.009000000000000005 3.743000000000052e-05 rpy=-6.4254155418928814e-15 -0.0 0.0 -> xyz=0.07402717 0.009000000000000005 3.743000000000052e-05 rpy=0 0 0
- joint l_hip_pitch_link_l_roll_joint: axis 1.0 0.0 -2.220446049246316e-16 -> 1.0 0 0; origin xyz=0.0 0.075 0.0012999999999999908 rpy=-1.5707963267948966 -1.5707963267948963 0 -> xyz=0 0.075 0.0012999999999999908 rpy=-1.5707963267948966 -1.5707963267948963 0
- joint l_hip_yaw_link_l_pitch_joint: axis 0.0 1.0 -1.222700479015263e-16 -> 0 1.0 0; origin xyz=-1.1048011099959547e-16 -0.07499999999999755 0.13630000000000136 rpy=1.2227004790152155e-16 1.5707963267948786 0 -> xyz=0 -0.07499999999999755 0.13630000000000136 rpy=0 1.5707963267948786 0
- joint l_shank_link_l_ankle_joint: axis -0.0 1.0 2.465190328815662e-32 -> 0 1.0 0; origin xyz=0.0 -0.3 -3.552713678800501e-17 rpy=1.5707963267948968 -0.0 0.0 -> xyz=0 -0.3 0 rpy=1.5707963267948968 0 0
- joint l_thigh_link_l_knee_joint: axis 0.0 1.2246467991536624e-16 -1.0 -> 0 0 -1.0; origin xyz=0.003499999999999997 -0.3 -0.013000000000000008 rpy=-1.2246467991481818e-16 -0.0 0.0 -> xyz=0.003499999999999997 -0.3 -0.013000000000000008 rpy=0 0 0
- joint pelvis_link_Rigid-31: origin xyz=-7.659717486428201e-12 -0.0004999999969337935 0.015 rpy=0.0 -0.0 -1.570796326794897 -> xyz=-7.659717486428201e-12 -0.0004999999969337935 0.015 rpy=0 0 -1.570796326794897
- joint pelvis_link_l_yaw_joint: axis 0.0 1.7918659470244052e-14 1.0 -> 0 0 1.0; origin xyz=0.11999999999233989 3.066148575681922e-12 -0.012 rpy=-3.1415926535897754 -0.0 -1.570796326794897 -> xyz=0.11999999999233989 3.066148575681922e-12 -0.012 rpy=-3.1415926535897754 0 -1.570796326794897
- joint pelvis_link_r_yaw_joint: axis 0.0 -1.7918659470244052e-14 -1.0 -> 0 0 -1.0; origin xyz=-0.12000000000765933 3.0662609857631655e-12 -0.012 rpy=-3.1415926535897754 -0.0 -1.570796326794897 -> xyz=-0.12000000000765933 3.0662609857631655e-12 -0.012 rpy=-3.1415926535897754 0 -1.570796326794897
- joint r_ankle_link_r_foot_joint: axis -1.0 0.0 2.16107724819376e-16 -> -1.0 0 0; origin xyz=0.07397279 0.009000000000000005 3.7410000000051014e-05 rpy=6.4254155418928814e-15 -0.0 0.0 -> xyz=0.07397279 0.009000000000000005 3.7410000000051014e-05 rpy=0 0 0
- joint r_hip_pitch_link_r_roll_joint: axis -1.0 0.0 2.220446049251407e-16 -> -1.0 0 0; origin xyz=0.0 -0.075 0.0013000000000000093 rpy=-1.5707963267948966 -1.5707963267948963 0 -> xyz=0 -0.075 0.0013000000000000093 rpy=-1.5707963267948966 -1.5707963267948963 0
- joint r_hip_yaw_link_r_pitch_joint: axis 0.0 1.0 -1.222700479015263e-16 -> 0 1.0 0; origin xyz=-1.1048011099959325e-16 0.07500000000000245 0.13629999999999867 rpy=1.2227004790152155e-16 1.5707963267948786 0 -> xyz=0 0.07500000000000245 0.13629999999999867 rpy=0 1.5707963267948786 0
- joint r_shank_link_r_ankle_joint: axis 0.0 -1.0 2.465190328815662e-32 -> 0 -1.0 0; origin xyz=0.0 -0.3 0.0 rpy=-1.5707963267948966 -0.0 0.0 -> xyz=0 -0.3 0 rpy=-1.5707963267948966 0 0
- joint r_thigh_link_r_knee_joint: axis 0.0 6.308915089505042e-28 -1.0 -> 0 0 -1.0; origin xyz=0.0035000000000000027 -0.3 0.013000000000000008 rpy=-8.689919168591649e-28 -0.0 0.0 -> xyz=0.0035000000000000027 -0.3 0.013000000000000008 rpy=0 0 0
- joint torso_link_imu_joint: origin xyz=-0.0338 0.036991 0.22879999 rpy=-1.5751289161869385e-15 -1.5707963267948966 0 -> xyz=-0.0338 0.036991 0.22879999 rpy=0 -1.5707963267948966 0

Commit message: replaced urdf

File: simulation/isaac/assets/robot/robot.urdf (robot description, URDF)
Before this commit: robot robot, 16 links, 15 joints
Links:
- link l_foot_link: mass 1.9784795442649168 -> 3.016240737310719
- link r_foot_link: mass 1.9784795442649097 -> 3.01624073731071
Joints:
- joint l_ankle_link_l_foot_joint: axis 1.0 0 0 -> 1.0 0.0 -2.16107724819376e-16; origin xyz=0.07402717 0.009000000000000005 3.743000000000052e-05 rpy=0 0 0 -> xyz=0.07402717 0.009000000000000005 3.743000000000052e-05 rpy=-6.4254155418928814e-15 -0.0 0.0
- joint l_hip_pitch_link_l_roll_joint: axis 1.0 0 0 -> 1.0 0.0 -2.220446049246316e-16; origin xyz=0 0.075 0.0012999999999999908 rpy=-1.5707963267948966 -1.5707963267948963 0 -> xyz=0.0 0.075 0.0012999999999999908 rpy=-1.5707963267948966 -1.5707963267948963 0
- joint l_hip_yaw_link_l_pitch_joint: axis 0 1.0 0 -> 0.0 1.0 -1.222700479015263e-16; origin xyz=0 -0.07499999999999755 0.13630000000000136 rpy=0 1.5707963267948786 0 -> xyz=-1.1048011099959547e-16 -0.07499999999999755 0.13630000000000136 rpy=1.2227004790152155e-16 1.5707963267948786 0
- joint l_shank_link_l_ankle_joint: axis 0 1.0 0 -> -0.0 1.0 2.465190328815662e-32; origin xyz=0 -0.3 0 rpy=1.5707963267948968 0 0 -> xyz=0.0 -0.3 -3.552713678800501e-17 rpy=1.5707963267948968 -0.0 0.0
- joint l_thigh_link_l_knee_joint: axis 0 0 -1.0 -> 0.0 1.2246467991536624e-16 -1.0; origin xyz=0.003499999999999997 -0.3 -0.013000000000000008 rpy=0 0 0 -> xyz=0.003499999999999997 -0.3 -0.013000000000000008 rpy=-1.2246467991481818e-16 -0.0 0.0
- joint pelvis_link_Rigid-31: origin xyz=-7.659717486428201e-12 -0.0004999999969337935 0.015 rpy=0 0 -1.570796326794897 -> xyz=-7.659717486428201e-12 -0.0004999999969337935 0.015 rpy=0.0 -0.0 -1.570796326794897
- joint pelvis_link_l_yaw_joint: axis 0 0 1.0 -> 0.0 1.7918659470244052e-14 1.0; origin xyz=0.11999999999233989 3.066148575681922e-12 -0.012 rpy=-3.1415926535897754 0 -1.570796326794897 -> xyz=0.11999999999233989 3.066148575681922e-12 -0.012 rpy=-3.1415926535897754 -0.0 -1.570796326794897
- joint pelvis_link_r_yaw_joint: axis 0 0 -1.0 -> 0.0 -1.7918659470244052e-14 -1.0; origin xyz=-0.12000000000765933 3.0662609857631655e-12 -0.012 rpy=-3.1415926535897754 0 -1.570796326794897 -> xyz=-0.12000000000765933 3.0662609857631655e-12 -0.012 rpy=-3.1415926535897754 -0.0 -1.570796326794897
- joint r_ankle_link_r_foot_joint: axis -1.0 0 0 -> -1.0 0.0 2.16107724819376e-16; origin xyz=0.07397279 0.009000000000000005 3.7410000000051014e-05 rpy=0 0 0 -> xyz=0.07397279 0.009000000000000005 3.7410000000051014e-05 rpy=6.4254155418928814e-15 -0.0 0.0
- joint r_hip_pitch_link_r_roll_joint: axis -1.0 0 0 -> -1.0 0.0 2.220446049251407e-16; origin xyz=0 -0.075 0.0013000000000000093 rpy=-1.5707963267948966 -1.5707963267948963 0 -> xyz=0.0 -0.075 0.0013000000000000093 rpy=-1.5707963267948966 -1.5707963267948963 0
- joint r_hip_yaw_link_r_pitch_joint: axis 0 1.0 0 -> 0.0 1.0 -1.222700479015263e-16; origin xyz=0 0.07500000000000245 0.13629999999999867 rpy=0 1.5707963267948786 0 -> xyz=-1.1048011099959325e-16 0.07500000000000245 0.13629999999999867 rpy=1.2227004790152155e-16 1.5707963267948786 0
- joint r_shank_link_r_ankle_joint: axis 0 -1.0 0 -> 0.0 -1.0 2.465190328815662e-32; origin xyz=0 -0.3 0 rpy=-1.5707963267948966 0 0 -> xyz=0.0 -0.3 0.0 rpy=-1.5707963267948966 -0.0 0.0
- joint r_thigh_link_r_knee_joint: axis 0 0 -1.0 -> 0.0 6.308915089505042e-28 -1.0; origin xyz=0.0035000000000000027 -0.3 0.013000000000000008 rpy=0 0 0 -> xyz=0.0035000000000000027 -0.3 0.013000000000000008 rpy=-8.689919168591649e-28 -0.0 0.0
- joint root: origin xyz=0 0 0.84 rpy=0 0 1.57079632679 -> xyz=0 0 0.85 rpy=0 0 1.57079632679
- joint torso_link_imu_joint: origin xyz=-0.0338 0.036991 0.22879999 rpy=0 -1.5707963267948966 0 -> xyz=-0.0338 0.036991 0.22879999 rpy=-1.5751289161869385e-15 -1.5707963267948966 0
